File: pmod-cp2104.sch (KiCad schematic (older format))
At the start: 37 parts, among them P1 PMOD-CONN_6X2, P2 USB_OTG, U1 CP2104

Commit message: Lots of small changes.
Parts:
- added CVD1: 1uF, Capacitors_SMD:C_0805, symbol C
- added DVD1: D, LEDs:LED_0402, symbol D
- added RDVD1: LEDO, Resistors_SMD:R_0603, symbol R
- added SW1: SW_PUSH, symbol SW_PUSH
- RUIO1, RUIO2, RUSP1: value 10k -> 4k7
Connections:
- net VUSB is gone; now on net CP_REGIN: P2.1 (VCC), U1.8 (VBUS)
- net CP_~RST: now also SW1.2
- net GND: now also CVD1.2, RDVD1.1, SW1.1
- net VDD: now also U1.6 (VDD), CVD1.1, DVD1.2 (A)
- new net: DVD1.1 (K), RDVD1.2
Other:
- note added: "DTR - Data Terminal Ready\n * USB -> Peripheral\n * Active Low\n * On Windows, DTR is held low while serial port is unopened\n\nFIXME: Wrong?\nMapping to PMOD_RST line"
- note added: "FIXME: Host here means??"
- note removed: "DTR - Data Terminal Ready\n * USB -> Peripheral\n * Active Low\n * On Windows, DTR is held low while serial port is unopened\n\nMapping to PMOD_RST line"
- moved on the sheet: RURST1
Changed lines of the file:
@@
 Text Notes 4000 2550 0    60   ~ 0
 VIO ==VPMOD\n Thus VPMOD always sets the IO voltage level\n\nREGIN - Regulator input - Feed from VUSB\n\nTake output at VDD to feed PMOD / VIO\n\n\nRegulator can supply 100mA output
-Text Label 5800 4400 1    60   ~ 0
+Text Label 5800 4450 1    60   ~ 0
 CP_~RST
 $Comp
 L R RURST1
 U 1 1 57F4DB18
-P 5800 3850
-F 0 "RURST1" V 5700 3850 50  0000 C CNN
-F 1 "4k7" V 5800 3850 50  0000 C CNN
-F 2 "Resistors_SMD:R_0603" V 5730 3850 50  0001 C CNN
-F 3 "" H 5800 3850 50  0000 C CNN
-	1    5800 3850
-	1    0    0    -1
-$EndComp
-Text Label 5800 3550 0    60   ~ 0
+P 5800 3800
+F 0 "RURST1" V 5700 3800 50  0000 C CNN
+F 1 "4k7" V 5800 3800 50  0000 C CNN
+F 2 "Resistors_SMD:R_0603" V 5730 3800 50  0001 C CNN
+F 3 "" H 5800 3800 50  0000 C CNN
+	1    5800 3800
+	1    0    0    -1
+$EndComp
+Text Label 5800 3500 0    60   ~ 0
 VIO
 $Comp
@@
 RI - Ring Indicator\n * Peripheral -> USB\n * Active Low\n * "Wake host up" signal\n\nMapping to PMOD_INT
 Text Notes 15050 5150 0    60   ~ 0
-DTR - Data Terminal Ready\n * USB -> Peripheral\n * Active Low\n * On Windows, DTR is held low while serial port is unopened\n\nMapping to PMOD_RST line
-Text Notes 17350 3150 0    60   ~ 0
+DTR - Data Terminal Ready\n * USB -> Peripheral\n * Active Low\n * On Windows, DTR is held low while serial port is unopened\n\nFIXME: Wrong?\nMapping to PMOD_RST line
+Text Notes 17350 3550 0    60   ~ 0
 DCD -- Data Carrier Detect\n * Peripheral -> USB\n * Active Low\n * On Linux, while DCD is low, nothing to do.
-Text Notes 15050 3150 0    60   ~ 0
+Text Notes 15050 3550 0    60   ~ 0
 DSR -- Data Set Ready\n * Peripheral -> USB\n * Active Low\n * Tied to DCD in "null modem" config.
 $Comp
@@
 Text Label 15050 5850 0    60   ~ 0
 PMOD_INT
-Text Notes 15050 3600 0    60   ~ 0
+Text Notes 15050 3050 0    60   ~ 0
 GPIO.3\n * USB->Peripheral\n * Active Low
-Text Notes 17350 3600 0    60   ~ 0
+Text Notes 17350 3050 0    60   ~ 0
 GPIO.2\n * USB->Peripheral\n * Active Low
 $Comp
@@
 P 17350 1200
 F 0 "RUIO1" V 17430 1200 50  0000 C CNN
-F 1 "10k" V 17350 1200 50  0000 C CNN
+F 1 "4k7" V 17350 1200 50  0000 C CNN
 F 2 "Resistors_SMD:R_0603" V 17280 1200 50  0001 C CNN
 F 3 "" H 17350 1200 50  0000 C CNN
@@
 P 16650 1200
 F 0 "RUIO2" V 16730 1200 50  0000 C CNN
-F 1 "10k" V 16650 1200 50  0000 C CNN
+F 1 "4k7" V 16650 1200 50  0000 C CNN
 F 2 "Resistors_SMD:R_0603" V 16580 1200 50  0001 C CNN
 F 3 "" H 16650 1200 50  0000 C CNN
@@
 P 3550 5300
 F 0 "RUSP1" V 3630 5300 50  0000 C CNN
-F 1 "10k" V 3550 5300 50  0000 C CNN
+F 1 "4k7" V 3550 5300 50  0000 C CNN
 F 2 "Resistors_SMD:R_0603" V 3480 5300 50  0001 C CNN
 F 3 "" H 3550 5300 50  0000 C CNN
@@
 	1    0    0    -1
 $EndComp
-Text Notes 3400 3150 0    60   ~ 0
+Text Notes 4650 3100 0    60   ~ 0
 UART Providing 3.3V power to PMOD Connector\nPMOD VCC <-- UART
 Text Label 17000 850  0    60   ~ 0
@@
 	2600 2600 2700 2600
 Wire Wire Line
-	2700 2600 2700 3050
-Wire Wire Line
-	2700 3050 1700 3050
+	2700 3050 2700 2600
+Wire Wire Line
+	1700 3050 2700 3050
 Wire Wire Line
 	1700 3050 1700 2600
@@
 Connection ~ 8400 5900
 Wire Wire Line
-	5800 4000 5800 4600
-Wire Wire Line
-	5800 3700 5800 3550
+	5800 3950 5800 4600
+Wire Wire Line
+	5800 3650 5800 3500
 Wire Wire Line
 	1750 5200 1900 5200
@@
 	6750 3800 6750 3900
 Wire Wire Line
-	6000 3800 6750 3800
+	6000 3800 7500 3800
 Wire Wire Line
 	17200 4150 17050 4150
@@
 	4100 2900 4400 2900
 Wire Wire Line
-	4400 2900 4400 2750
+	4400 2750 4400 3200
 Wire Wire Line
 	16850 900  17150 900
@@
 	7500 3600 7500 5200
 Wire Wire Line
-	5500 4600 5500 4400
-Wire Wire Line
-	5500 4400 4250 4400
-Wire Wire Line
-	5600 4600 5600 4300
-Wire Wire Line
-	5600 4300 4250 4300
-Text Label 4250 4400 0    60   ~ 0
+	5500 4600 5500 4550
+Wire Wire Line
+	5500 4550 4250 4550
+Wire Wire Line
+	5600 4600 5600 4450
+Wire Wire Line
+	5600 4450 4250 4450
+Text Label 4250 4550 0    60   ~ 0
 CP_GPIO.2
-Text Label 4250 4300 0    60   ~ 0
+Text Label 4250 4450 0    60   ~ 0
 CP_GPIO.3
 Wire Wire Line
@@
 	1    0    0    -1
 $EndComp
+Wire Wire Line
+	6500 5100 6900 5100
+Text Label 6900 5100 0    60   ~ 0
+VDD
+$Comp
+L D DVD1
+U 1 1 57F636FC
+P 4400 3350
+F 0 "DVD1" H 4400 3450 50  0000 C CNN
+F 1 "D" H 4400 3250 50  0001 C CNN
+F 2 "LEDs:LED_0402" H 4400 3350 50  0001 C CNN
+F 3 "" H 4400 3350 50  0000 C CNN
+	1    4400 3350
+	0    1    -1   0
+$EndComp
+$Comp
+L R RDVD1
+U 1 1 57F63702
+P 4400 3800
+F 0 "RDVD1" V 4480 3800 50  0000 C CNN
+F 1 "LEDO" V 4400 3800 50  0000 C CNN
+F 2 "Resistors_SMD:R_0603" V 4330 3800 50  0001 C CNN
+F 3 "" H 4400 3800 50  0000 C CNN
+	1    4400 3800
+	1    0    0    1
+$EndComp
+Wire Wire Line
+	4400 3950 4400 4050
+Wire Wire Line
+	4400 3650 4400 3500
+$Comp
+L GND #PWR?
+U 1 1 57F63A8D
+P 4400 4050
+F 0 "#PWR?" H 4400 3800 50  0001 C CNN
+F 1 "GND" H 4400 3900 50  0000 C CNN
+F 2 "" H 4400 4050 50  0000 C CNN
+F 3 "" H 4400 4050 50  0000 C CNN
+	1    4400 4050
+	-1   0    0    -1
+$EndComp
+Connection ~ 4400 2900
+$Comp
+L C CVD1
+U 1 1 57F6453F
+P 4150 3650
+F 0 "CVD1" H 4175 3750 50  0000 L CNN
+F 1 "1uF" H 4175 3550 50  0000 L CNN
+F 2 "Capacitors_SMD:C_0805" H 4188 3500 50  0001 C CNN
+F 3 "" H 4150 3650 50  0000 C CNN
+	1    4150 3650
+	-1   0    0    -1
+$EndComp
+Wire Wire Line
+	4150 3500 4150 2900
+Connection ~ 4150 2900
+Wire Wire Line
+	4150 4000 5050 4000
+Wire Wire Line
+	4150 4000 4150 3800
+Connection ~ 4400 4000
+Connection ~ 7500 3800
+Connection ~ 6750 3800
+Text Notes 14950 4150 2    60   ~ 0
+Out >
+Text Notes 14950 5700 2    60   ~ 0
+In <
+Text Notes 3200 1000 0    60   ~ 0
+FIXME: Host here means??
+$Comp
+L SW_PUSH SW1
+U 1 1 57F6685A
+P 5350 4000
+F 0 "SW1" H 5500 4110 50  0000 C CNN
+F 1 "SW_PUSH" H 5350 3920 50  0000 C CNN
+F 2 "" H 5350 4000 50  0000 C CNN
+F 3 "" H 5350 4000 50  0000 C CNN
+	1    5350 4000
+	1    0    0    -1
+$EndComp
+Wire Wire Line
+	5650 4000 5800 4000
+Connection ~ 5800 4000
 $EndSCHEMATC

Commit message: Making everything fit on one sheet.
Parts:
- SW1: footprint (none) -> Buttons_Switches_SMD:SW_SPST_PTS645
Other:
- moved on the sheet: CREGIN1, CVD1, CVPP1, DDTR1, DIO1, DIO2, DRI1, DRX1, DSP1, DTX1, DVD1, JPDTR1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
